Commit message: fix-diff wheel continous xacro now working (need JSP on dockerfile from #10)

File: warrior1_description/xacro/diff_wheel.xacro (robot description, xacro)
@@ -1,27 +1,36 @@
 <?xml version="1.0"?>
-<robot xmlns:xacro="http://www.ros.org/wiki/xacro" >
-<xacro:macro name="wheel" params="prefix parent_link x y z roll pitch yaw">
-    <joint name="${prefix}_wheel_joint" type="continuous">
-        <parent link="{parent_link}"/>
-        <child link="${prefix}_wheel"/>
-        <origin xyz="${x} ${y} ${z}" rpy="${roll} ${pitch} ${yaw}"/>
-        <axis xyz="0 0 0"/>
-    </joint>
-    <link name="${prefix}_wheel">
-    <visual>
-        <geometry>
-            <cylinder length="${diff_wheel_width}" radius="${diff_wheel_radius}" />
-        </geometry>
-        <material name="blue"/>
-    </visual>
-    <collision>
-        <geometry>
-            <cylinder length="${diff_wheel_width}" radius="${diff_wheel_radius}" />
-        </geometry>
-    </collision>
-    <xacro:inertial_cylinder mass="0.1" length="0.05" radius="0.05">
-        <origin xyz="${x} ${y} ${z}" rpy="${roll} ${pitch} ${yaw}"/>
-    </xacro:inertial_cylinder>
-    </link>
-</xacro:macro>
+<robot xmlns:xacro="http://www.ros.org/wiki/xacro">
+    <xacro:macro name="diff_wheel"
+                 params="prefix parent_link x y z roll pitch yaw">
+        <joint name="${prefix}_wheel_joint" type="continuous">
+            <parent link="base_link"/>
+            <child link="${prefix}_wheel"/>
+            <origin xyz="${x} ${y} ${z}"
+                    rpy="${roll} ${pitch} ${yaw}"/>
+            <axis xyz="0 0 1"/>
+        </joint>
+        <link name="${prefix}_wheel">
+            <visual>
+                <geometry>
+                    <cylinder
+                        length="${diff_wheel_width}"
+                        radius="${diff_wheel_radius}"/>
+                </geometry>
+                <material name="blue"/>
+            </visual>
+            <collision>
+                <geometry>
+                    <cylinder
+                        length="${diff_wheel_width}"
+                        radius="${diff_wheel_radius}"/>
+                </geometry>
+            </collision>
+            <xacro:inertial_cylinder
+                mass="0.1"
+                length="${diff_wheel_width}"
+                radius="${diff_wheel_radius}">
+                <origin xyz="0 0 0" rpy="0 0 0"/>
+            </xacro:inertial_cylinder>
+        </link>
+    </xacro:macro>
 </robot>
